File: 12VSB.kicad_sch (KiCad schematic)
At the start: 24 parts

Commit message: initial pcb dump
Parts:
- C1, C2, C5, C6: footprint (none) -> Capacitor_SMD:C_0805_2012Metric
- C10, C4: footprint (none) -> Capacitor_SMD:C_0402_1005Metric
- C12, C3, C9: footprint (none) -> Capacitor_SMD:C_0603_1608Metric
- D1, D2: value (none) -> SH548F; footprint Diode_THT:D_DO-35_SOD27_P7.62mm_Horizontal -> 12VSB Library:diode
- H1, H2, H3, H4: footprint (none) -> MountingHole:MountingHole_3.5mm_Pad
- L1: value L -> L 3R3; footprint (none) -> 12VSB Library:INDM125125X800N
- R1, R2, R3, R4: footprint (none) -> Resistor_SMD:R_0402_1005Metric
- R10, R5, R8: footprint (none) -> Resistor_SMD:R_0603_1608Metric
- U1: value ~ -> FP6296
Other:
- note added: "5VSB to 12VSB Adapter"
- moved on the sheet: C1, C10, C12, C2, C3, C4, C5, C6, C9, D1, D2, H1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

Commit message: updated pcb layout
Parts:
- H1, H2, H3, H4: footprint MountingHole:MountingHole_3.5mm_Pad -> MountingHole:MountingHole_2.2mm_M2_DIN965_Pad
Changed lines of the file:
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@@
       (effects (font (size 1.27 1.27)))
     )
-    (property "Footprint" "MountingHole:MountingHole_3.5mm_Pad" (at 26.67 73.66 0)
+    (property "Footprint" "MountingHole:MountingHole_2.2mm_M2_DIN965_Pad" (at 26.67 73.66 0)
       (effects (font (size 1.27 1.27)) hide)
     )
@@
       (effects (font (size 1.27 1.27)))
     )
-    (property "Footprint" "MountingHole:MountingHole_3.5mm_Pad" (at 26.67 64.77 0)
+    (property "Footprint" "MountingHole:MountingHole_2.2mm_M2_DIN965_Pad" (at 26.67 64.77 0)
       (effects (font (size 1.27 1.27)) hide)
     )
@@
       (effects (font (size 1.27 1.27)) hide)
     )
-    (property "Datasheet" "https://www.microsemi.com/document-portal/doc_download/8865-lds-0040-datasheet" (at 71.12 97.79 0)
+    (property "Datasheet" "" (at 71.12 97.79 0)
       (effects (font (size 1.27 1.27)) hide)
     )
@@
       (effects (font (size 1.27 1.27)))
     )
-    (property "Footprint" "MountingHole:MountingHole_3.5mm_Pad" (at 26.67 82.55 0)
+    (property "Footprint" "MountingHole:MountingHole_2.2mm_M2_DIN965_Pad" (at 26.67 82.55 0)
       (effects (font (size 1.27 1.27)) hide)
     )
@@
       (effects (font (size 1.27 1.27)) hide)
     )
-    (property "Datasheet" "https://www.microsemi.com/document-portal/doc_download/8865-lds-0040-datasheet" (at 60.96 22.86 0)
+    (property "Datasheet" "" (at 60.96 22.86 0)
       (effects (font (size 1.27 1.27)) hide)
     )
@@
       (effects (font (size 1.27 1.27)))
     )
-    (property "Footprint" "MountingHole:MountingHole_3.5mm_Pad" (at 26.67 93.98 0)
-      (effects (font (size 1.27 1.27)) hide)
-    )
+    (property "Footprint" "MountingHole:MountingHole_2.2mm_M2_DIN965_Pad" (at 26.67 93.98 0)
+      (effects (font (size 1.27 1.27)) hide)
+    )

Commit message: Corrected Schema and updated PCB Layout
Parts:
- L1: symbol Device:L -> Device:L_Iron
Connections:
- net GNDREF renamed GND
Other:
- moved on the sheet: C10, C12, C4, C9, R3, R4, R5, R8

Commit message: Updated PCB Layout and Documentation
Parts:
- D1, D2: value SH548F -> SH54BF
Changed lines of the file:
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@@
       (effects (font (size 1.27 1.27)))
     )
-    (property "Value" "SH548F" (at 71.4375 95.4311 0)
+    (property "Value" "SH54BF" (at 71.4375 95.4311 0)
       (effects (font (size 1.27 1.27)))
     )
@@
       (effects (font (size 1.27 1.27)))
     )
-    (property "Value" " SH548F" (at 61.2775 20.5011 0)
-      (effects (font (size 1.27 1.27)))
-    )
+    (property "Value" " SH54BF" (at 61.2775 20.5011 0)
+      (effects (font (size 1.27 1.27)))
+    )
