File: 12VSB.kicad_sch (KiCad schematic)
At the start: 24 parts, among them U1 FP6296

Commit message: corrected schematic
Parts:
- R1: value R 30D -> 200K
- R10: value R 102 -> 1K
- R2: value R 223 -> 22K
- R3: value R 01D -> 100K
- R4: value R 303 -> 30K
- R5: value R -> 100
- R8: value R 1R5 -> 1.5
Changed lines of the file:
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@@
       (effects (font (size 1.27 1.27)) (justify left))
     )
-    (property "Value" "R 30D" (at 123.698 31.7573 0)
+    (property "Value" "200K" (at 123.698 31.7573 0)
       (effects (font (size 1.27 1.27)) (justify left))
     )
@@
       (effects (font (size 1.27 1.27)))
     )
-    (property "Value" "R 102" (at 41.91 47.4251 90)
+    (property "Value" "1K" (at 41.91 47.4251 90)
       (effects (font (size 1.27 1.27)))
     )
@@
       (effects (font (size 1.27 1.27)))
     )
-    (property "Value" "R 1R5" (at 41.91 30.9151 90)
+    (property "Value" "1.5" (at 41.91 30.9151 90)
       (effects (font (size 1.27 1.27)))
     )
@@
       (effects (font (size 1.27 1.27)) (justify left))
     )
-    (property "Value" "R" (at 76.708 27.9473 0)
+    (property "Value" "100" (at 76.708 27.9473 0)
       (effects (font (size 1.27 1.27)) (justify left))
     )
@@
       (effects (font (size 1.27 1.27)))
     )
-    (property "Value" "R 01D" (at 91.44 38.5351 90)
+    (property "Value" "100K" (at 91.44 38.5351 90)
       (effects (font (size 1.27 1.27)))
     )
@@
       (effects (font (size 1.27 1.27)) (justify left))
     )
-    (property "Value" "R 223" (at 123.698 41.9173 0)
+    (property "Value" "22K" (at 123.698 41.9173 0)
       (effects (font (size 1.27 1.27)) (justify left))
     )
@@
       (effects (font (size 1.27 1.27)))
     )
-    (property "Value" "R 303" (at 80.01 46.1551 90)
-      (effects (font (size 1.27 1.27)))
-    )
+    (property "Value" "30K" (at 80.01 46.1551 90)
+      (effects (font (size 1.27 1.27)))
+    )

Commit message: Updated schematic
Parts:
- C1, C2, C5, C6: value C 22uF -> 22uF
- C10: value C -> 470pF
- C12: value C 1nF -> 1nF
- C3: value C 1uF -> 1uF
- C4: value C -> 2.2nF
- C9: value C 0.1uF -> 0.1uF
Changed lines of the file:
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@@
       (effects (font (size 1.27 1.27)))
     )
-    (property "Value" "C 1nF" (at 31.75 29.7721 90)
+    (property "Value" "1nF" (at 31.75 29.7721 90)
       (effects (font (size 1.27 1.27)))
     )
@@
       (effects (font (size 1.27 1.27)) (justify left))
     )
-    (property "Value" "C 22uF" (at 86.741 68.5873 0)
+    (property "Value" "22uF" (at 86.741 68.5873 0)
       (effects (font (size 1.27 1.27)) (justify left))
     )
@@
       (effects (font (size 1.27 1.27)))
     )
-    (property "Value" "C" (at 91.44 45.0121 90)
+    (property "Value" "2.2nF" (at 91.44 45.0121 90)
       (effects (font (size 1.27 1.27)))
     )
@@
       (effects (font (size 1.27 1.27)))
     )
-    (property "Value" "C 1uF" (at 41.91 37.3921 90)
+    (property "Value" "1uF" (at 41.91 37.3921 90)
       (effects (font (size 1.27 1.27)))
     )
@@
       (effects (font (size 1.27 1.27)) (justify left))
     )
-    (property "Value" "C 22uF" (at 86.741 85.0973 0)
+    (property "Value" "22uF" (at 86.741 85.0973 0)
       (effects (font (size 1.27 1.27)) (justify left))
     )
@@
       (effects (font (size 1.27 1.27)) (justify left))
     )
-    (property "Value" "C 22uF" (at 71.501 68.5873 0)
+    (property "Value" "22uF" (at 71.501 68.5873 0)
       (effects (font (size 1.27 1.27)) (justify left))
     )
@@
       (effects (font (size 1.27 1.27)))
     )
-    (property "Value" "C" (at 91.44 53.9021 90)
+    (property "Value" "470pF" (at 91.44 53.9021 90)
       (effects (font (size 1.27 1.27)))
     )
@@
       (effects (font (size 1.27 1.27)))
     )
-    (property "Value" " C 0.1uF" (at 91.44 29.7721 90)
+    (property "Value" "0.1uF" (at 91.44 29.7721 90)
       (effects (font (size 1.27 1.27)))
     )
@@
       (effects (font (size 1.27 1.27)) (justify left))
     )
-    (property "Value" "C 22uF" (at 71.501 85.0973 0)
-      (effects (font (size 1.27 1.27)) (justify left))
-    )
+    (property "Value" "22uF" (at 71.501 85.0973 0)
+      (effects (font (size 1.27 1.27)) (justify left))
+    )
